Commit message: fabo_shell和fake_nav 已添加

File: my_gazebo/urdf/kinectv1_neck.urdf.xacro (robot description, xacro)
@@ -47,4 +47,7 @@
     </gazebo>
   </xacro:macro>
+  <!-- kinect 旧版本 -->
+  <xacro:include filename="$(find my_gazebo)/urdf/kinect.urdf.xacro"/>
+  <!-- kinectv1 huxianxu版本 -->
   <xacro:macro name="kinectv1" params="parent">
       <joint name="camera_rgb_joint" type="fixed">
@@ -110,4 +113,5 @@
       <xacro:sim_3dcamera/>
   </xacro:macro>
+  <!-- 添加脖子 -->
   <xacro:macro name="kinectv1_neck" params="parent camera_offset_x camera_offset_y camera_offset_z">
         <joint name="joint_neck_1" type="revolute">
@@ -139,5 +143,5 @@
         </link>
         <joint name="joint_neck_2" type="fixed">
-          <origin xyz="0.0 0.0 0.1" rpy="0 0.4887 0"/>
+          <origin xyz="0.0 0.0 0.0" rpy="0 0.4887 0"/>   <!-- 28 angle 0.4887hudu -->
           <parent link="platform_1"/>
           <child link="platform_2"/>
@@ -163,5 +167,6 @@
         </link>
         <!-- rplidar sensor for simulation -->
-        <xacro:kinectv1 parent="platform_2" />
+        <!-- <xacro:kinectv1 parent="platform_2" /> -->
+        <xacro:sensor_kinect parent="platform_2"/>
         <transmission name="transmission_neck">
           <type>transmission_interface/SimpleTransmission</type>

File: my_gazebo/urdf/robot_hokuyo_kinectv1neck.urdf.xacro (robot description, xacro)
@@ -13,5 +13,5 @@
 	<xacro:property name="camera_offset_x" value="0.0" />
 	<xacro:property name="camera_offset_y" value="0.0" />
-	<xacro:property name="camera_offset_z" value="0.9" />
-	<xacro:kinectv1_neck parent="plate_2_link" camera_offset_x="${camera_offset_x}" camera_offset_y="${camera_offset_y}" camera_offset_z="${camera_offset_z}" />
+	<xacro:property name="camera_offset_z" value="1.2" />
+	<xacro:kinectv1_neck parent="base_footprint" camera_offset_x="${camera_offset_x}" camera_offset_y="${camera_offset_y}" camera_offset_z="${camera_offset_z}" />
 </robot>

File: my_gazebo/urdf/test_robot_body.urdf.xacro (robot description, xacro)
@@ -27,5 +27,5 @@
     <xacro:property name="caster_radius"          value="0.016" />
     <xacro:property name="caster_mass"            value="0.01" />
-    <xacro:property name="caster_joint_origin_x"  value="-0.25" />
+    <xacro:property name="caster_joint_origin_x"  value="-0.2" />
     <!-- Wheel radius, height and mass -->
     <xacro:property name="wheel_radius" value="0.033" />
@@ -239,5 +239,5 @@
                 rpy="0 0 0" />
             <mass
-                value="0.0000000000000001" />
+                value="1e-5" />
             <inertia
                 ixx="0.172898160476508"
@@ -254,5 +254,5 @@
             <geometry>
                 <mesh
-                filename="package://fabo_shell/meshes/shell_link.STL" />
+                filename="package://my_gazebo/urdf/shell_link.STL" />
             </geometry>
             <material
@@ -268,5 +268,5 @@
             <geometry>
                 <mesh
-                filename="package://fabo_shell/meshes/shell_link.STL" />
+                filename="package://my_gazebo/urdf/shell_link.STL" />
             </geometry>
             </collision>
