Commit message: GlobalPlanner DWA

File: my_gazebo/urdf/test_robot_body.urdf.xacro (robot description, xacro)
@@ -21,5 +21,5 @@
     <!-- Main body length, width, height and mass -->
     <xacro:property name="base_mass"        value="0.5" />
-    <xacro:property name="base_link_radius" value="0.2"/>   <!-- 原： 0.13 -->
+    <xacro:property name="base_link_radius" value="0.13"/>   <!-- origin: 0.13   fabo:0.2-->
     <xacro:property name="base_link_length" value="0.005"/>
     <xacro:property name="motor_x" value="0"/>
@@ -27,5 +27,5 @@
     <xacro:property name="caster_radius"          value="0.016" />
     <xacro:property name="caster_mass"            value="0.01" />
-    <xacro:property name="caster_joint_origin_x"  value="-0.2" />
+    <xacro:property name="caster_joint_origin_x"  value="-0.13" />    <!-- caster position to center.  fabo:0.2     -->
     <!-- Wheel radius, height and mass -->
     <xacro:property name="wheel_radius" value="0.033" />
@@ -267,6 +267,6 @@
                 rpy="0 0 0" />
             <geometry>
-                <mesh
-                filename="package://my_gazebo/urdf/shell_link.STL" />
+                <cylinder length="${base_link_length}" radius="${base_link_radius}"/>
+                <!-- <mesh   filename="package://my_gazebo/urdf/shell_link.STL" /> -->
             </geometry>
             </collision>
