Commit message: continus的neck关节中添加velocity=1；增加了新的物体布局

File: my_gazebo/urdf/kinect.urdf.xacro (robot description, xacro)
@@ -6,5 +6,5 @@
       <sensor type="depth" name="camera">
         <always_on>true</always_on>
-        <update_rate>20.0</update_rate>
+        <update_rate>30.0</update_rate>
         <camera>
           <horizontal_fov>${60.0*M_PI/180.0}</horizontal_fov>
@@ -22,5 +22,5 @@
           <cameraName>/</cameraName>
           <alwaysOn>true</alwaysOn>
-          <updateRate>10</updateRate>
+          <updateRate>30</updateRate>
           <imageTopicName>rgb/image_raw</imageTopicName>
           <depthImageTopicName>/depth_to_rgb/image_raw</depthImageTopicName>

File: my_gazebo/urdf/kinectv1_neck.urdf.xacro (robot description, xacro)
@@ -115,11 +115,13 @@
   <!-- 添加脖子 -->
   <xacro:macro name="kinectv1_neck" params="parent camera_offset_x camera_offset_y camera_offset_z">
-        <joint name="joint_neck_1" type="revolute">
+        <!-- <joint name="joint_neck_1" type="revolute">  -->
+        <joint name="joint_neck_1" type="continuous">
           <origin xyz="${camera_offset_x} ${camera_offset_y} ${camera_offset_z}" rpy="0 0 0"/>
           <parent link="${parent}"/>
           <child link="platform_1"/>
           <axis xyz="0 0 1"/>
-          <limit effort="300" velocity="1" lower="-1.57" upper="1.57"/>
-          <dynamics damping="50" friction="1"/>
+          <limit effort="300" velocity="1" lower="-3.14" upper="3.14"/>
+          <!-- 1.57  M_PI-->
+          <dynamics damping="0.1" friction="0.5"/><!-- <dynamics damping="50" friction="1"/> -->
         </joint>
         <link name="platform_1">

File: my_gazebo/urdf/robot_hokuyo_kinectv1neck.urdf.xacro (robot description, xacro)
@@ -13,5 +13,5 @@
 	<xacro:property name="camera_offset_x" value="0.0" />
 	<xacro:property name="camera_offset_y" value="0.0" />
-	<xacro:property name="camera_offset_z" value="1.2" />
+	<xacro:property name="camera_offset_z" value="1.4" />
 	<xacro:kinectv1_neck parent="base_footprint" camera_offset_x="${camera_offset_x}" camera_offset_y="${camera_offset_y}" camera_offset_z="${camera_offset_z}" />
 </robot>
