Commit message: 重新梳理

File: ASLAM_gazebo_world/urdf/hokuyo.urdf.xacro (robot description, xacro)
@@ -1,6 +1,6 @@
 <?xml version="1.0"?>
     <robot name="laser_hokuyo" xmlns:xacro="http://ros.org/wiki/xacro">
-      <!-- <xacro:include filename="$(find my_gazebo)/urdf/turtlebot_thirdparty/turtlebot_gazebo.urdf.xacro"/>   -->
-      <!-- <xacro:include filename="$(find my_gazebo)/urdf/turtlebot_thirdparty/turtlebot_properties.urdf.xacro"/>   -->
+      <!-- <xacro:include filename="$(find ASLAM_gazebo_world)/urdf/turtlebot_thirdparty/turtlebot_gazebo.urdf.xacro"/>   -->
+      <!-- <xacro:include filename="$(find ASLAM_gazebo_world)/urdf/turtlebot_thirdparty/turtlebot_properties.urdf.xacro"/>   -->
       <!-- Set up laser gazebo details -->
       <xacro:macro name="sim_hokuyo_range_finder">

File: ASLAM_gazebo_world/urdf/kinect.urdf.xacro (robot description, xacro)
@@ -72,5 +72,5 @@
         <geometry>
          <!-- <mesh filename="package://turtlebot_description/meshes/sensors/kinect.dae"/> -->
-         <mesh filename="$(find my_gazebo)/urdf/kinect.dae"/>
+         <mesh filename="$(find ASLAM_gazebo_world)/urdf/kinect.dae"/>
         </geometry>
       </visual>

File: ASLAM_gazebo_world/urdf/kinectv1_neck.urdf.xacro (robot description, xacro)
@@ -48,5 +48,5 @@
   </xacro:macro>
   <!-- kinect 旧版本 -->
-  <xacro:include filename="$(find my_gazebo)/urdf/kinect.urdf.xacro"/>
+  <xacro:include filename="$(find ASLAM_gazebo_world)/urdf/kinect.urdf.xacro"/>
   <!-- kinectv1 huxianxu版本 -->
   <xacro:macro name="kinectv1" params="parent">
@@ -78,5 +78,5 @@
           <origin xyz="0 0 0" rpy="0 0 ${M_PI/2}"/>
           <geometry>
-            <mesh filename="package://my_gazebo/urdf/kinect.dae"/>
+            <mesh filename="package://ASLAM_gazebo_world/urdf/kinect.dae"/>
           </geometry>
         </visual>

File: ASLAM_gazebo_world/urdf/robot_hokuyo_kinectv1neck.urdf copy.xacro (robot description, xacro)
@@ -2,13 +2,13 @@
 <robot name="mrobot" xmlns:xacro="http://www.ros.org/wiki/xacro">
 <!-- robot_mrobot/mrobot_gazebo/urdf/dianzikeji -->
-    <xacro:include filename="$(find my_gazebo)/urdf/test_robot.urdf.xacro" />
-    <!-- <xacro:include filename="$(find my_gazebo)/urdf/test_arm.xacro" /> -->
+    <xacro:include filename="$(find ASLAM_gazebo_world)/urdf/test_robot.urdf.xacro" />
+    <!-- <xacro:include filename="$(find ASLAM_gazebo_world)/urdf/test_arm.xacro" /> -->
     <!-- 雷达hokuyo --><!-- 相机kinectv1 -->
-    <!-- <xacro:include filename="$(find my_gazebo)/urdf/hokuyo.urdf.xacro" />
+    <!-- <xacro:include filename="$(find ASLAM_gazebo_world)/urdf/hokuyo.urdf.xacro" />
 	<xacro:property name="laser_offset_x" value="0.2" />
 	<xacro:property name="laser_offset_y" value="0" />
 	<xacro:property name="laser_offset_z" value="-0.1" />
 	<xacro:laser_hokuyo parent="plate_2_link" laser_offset_x="${laser_offset_x}" laser_offset_y="${laser_offset_y}" laser_offset_z="${laser_offset_z}" />
-    <xacro:include filename="$(find my_gazebo)/urdf/kinectv1_neck.urdf.xacro" />
+    <xacro:include filename="$(find ASLAM_gazebo_world)/urdf/kinectv1_neck.urdf.xacro" />
 	<xacro:property name="camera_offset_x" value="0.0" />
 	<xacro:property name="camera_offset_y" value="0.0" />

File: ASLAM_gazebo_world/urdf/robot_hokuyo_kinectv1neck.urdf.xacro (robot description, xacro)
@@ -2,7 +2,7 @@
 <robot name="mrobot" xmlns:xacro="http://www.ros.org/wiki/xacro">
 <!-- robot_mrobot/mrobot_gazebo/urdf/dianzikeji -->
-    <xacro:include filename="$(find my_gazebo)/urdf/test_robot.urdf.xacro" />
+    <xacro:include filename="$(find ASLAM_gazebo_world)/urdf/test_robot.urdf.xacro" />
 	<!-- 雷达hokuyo -->
-    <xacro:include filename="$(find my_gazebo)/urdf/hokuyo.urdf.xacro" />
+    <xacro:include filename="$(find ASLAM_gazebo_world)/urdf/hokuyo.urdf.xacro" />
 	<xacro:property name="laser_offset_x" value="0.25" />  <!-- 原： 0.1 -->
 	<xacro:property name="laser_offset_y" value="0" />
@@ -10,5 +10,5 @@
 	<xacro:laser_hokuyo parent="plate_2_link" laser_offset_x="${laser_offset_x}" laser_offset_y="${laser_offset_y}" laser_offset_z="${laser_offset_z}" />
 	<!-- 相机kinectv1 -->
-	<xacro:include filename="$(find my_gazebo)/urdf/kinectv1_neck.urdf.xacro" />
+	<xacro:include filename="$(find ASLAM_gazebo_world)/urdf/kinectv1_neck.urdf.xacro" />
 	<xacro:property name="camera_offset_x" value="0.0" />
 	<xacro:property name="camera_offset_y" value="0.0" />

File: ASLAM_gazebo_world/urdf/test_robot.urdf.xacro (robot description, xacro)
@@ -1,5 +1,5 @@
 <?xml version="1.0"?>
 <robot name="mrobot" xmlns:xacro="http://www.ros.org/wiki/xacro">
-	<xacro:include filename="$(find my_gazebo)/urdf/test_robot_body.urdf.xacro" />
+	<xacro:include filename="$(find ASLAM_gazebo_world)/urdf/test_robot_body.urdf.xacro" />
 	<!-- Body of mrobot, with plates, standoffs -->
 	<mrobot_body/>

File: ASLAM_gazebo_world/urdf/test_robot_body.urdf.xacro (robot description, xacro)
@@ -254,5 +254,5 @@
             <geometry>
                 <mesh
-                filename="package://my_gazebo/urdf/shell_link.STL" />
+                filename="package://ASLAM_gazebo_world/urdf/shell_link.STL" />
             </geometry>
             <material
@@ -268,5 +268,5 @@
             <geometry>
                 <cylinder length="${base_link_length}" radius="${base_link_radius}"/>
-                <!-- <mesh   filename="package://my_gazebo/urdf/shell_link.STL" /> -->
+                <!-- <mesh   filename="package://ASLAM_gazebo_world/urdf/shell_link.STL" /> -->
             </geometry>
             </collision>

File: ASLAM_gazebo_world/urdf/test_robot_rplidar_neck.xacro (robot description, xacro)
@@ -2,6 +2,6 @@
 <robot name="mrobot" xmlns:xacro="http://www.ros.org/wiki/xacro">
 <!-- robot_mrobot/mrobot_gazebo/urdf/dianzikeji -->
-    <xacro:include filename="$(find my_gazebo)/urdf/test_robot.urdf.xacro" />
-    <xacro:include filename="$(find my_gazebo)/urdf/test_arm.xacro" />
+    <xacro:include filename="$(find ASLAM_gazebo_world)/urdf/test_robot.urdf.xacro" />
+    <xacro:include filename="$(find ASLAM_gazebo_world)/urdf/test_arm.xacro" />
     <xacro:property name="offset_x" value="0.03" />
     <xacro:property name="offset_y" value="0" />
@@ -13,5 +13,5 @@
     </joint>
     <!-- 雷达 -->
-    <xacro:include filename="$(find my_gazebo)/urdf/test_rplidar.xacro" />
+    <xacro:include filename="$(find ASLAM_gazebo_world)/urdf/test_rplidar.xacro" />
 	<xacro:property name="rplidar_offset_x" value="0" />
 	<xacro:property name="rplidar_offset_y" value="0" />
